File: pcb/microcontroller.brd (EAGLE design)
At the start: 31.1 x 30.9 mm, 8 parts

Commit message: microcontroller board ready to be fab'd
Parts:
- moved JP1 57.0 mm to (24.5, 13.1), turned to 90 degrees
- moved JP2 46.6 mm to (1.65, 13.1), turned to 270 degrees
- moved R13 24.2 mm to (4.70, 2.41), turned to 180 degrees
- moved R11 18.7 mm to (22.4, 22.2)
- moved C10 12.1 mm to (19.6, 2.41)
- moved R12 7.51 mm to (9.40, 2.41), turned to 180 degrees
- moved X1 4.99 mm to (13.0, 14.7), turned to 0 degrees
- moved R10 4.47 mm to (14.1, 2.41), turned to 0 degrees
Connections:
- removed net N$2: X1.6
- net A0: now also X1.2
- net D6/GPIO12: now also X1.6
Routing:
- net +3V3: track 0.00 -> 38.9 mm, vias 0 -> 2
- net D8/GPIO15: track 0.00 -> 26.0 mm, vias 0 -> 1
- net CH_PD: track 0.00 -> 16.7 mm
- net D3/GPIO0: track 0.00 -> 14.9 mm
- net D2/GPIO4: track 0.00 -> 9.43 mm
- net RESET: track 0.00 -> 7.46 mm
- net D0/GPIO16: track 0.00 -> 6.32 mm
- net D1/GPIO5: track 0.00 -> 6.09 mm
- net D5/GPIO14/SCK: track 0.00 -> 5.79 mm
- net D6/GPIO12: track 0.00 -> 5.21 mm
- net TX: track 0.00 -> 5.17 mm
- net A0: track 0.00 -> 5.05 mm
- net D7/GPIO13/MOSI: track 0.00 -> 5.00 mm
- net RX: track 0.00 -> 4.70 mm
- net D4/GPIO2: track 0.00 -> 3.81 mm
Other:
- board size 31.1 x 30.9 mm -> 26.2 x 26.2 mm
