File: pcb/microcontroller.brd (EAGLE design)
At the start: 26.2 x 26.2 mm, 15 parts, among them J1 SMD, U1 MMA8452Q

Commit message: Fix header direction on microcontroller board
Parts:
- flipped JP1 to the bottom
- flipped JP2 to the bottom
