File: pcb/oled.sch (EAGLE design)
At the start: 20 parts, among them U1 UG-2828GDEDF11, U2 FAN5331SX

Commit message: Use cheaper 0.1uF capacitors and 10uF capacitors
Parts:
- C2, C3, C4, C6: MPN EMK212ABJ106KG-T -> LMK212BJ106KG-T
- C7: MPN 08051C104J4T4A -> C0805C104M3RACTU
Changed lines of the file:
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@@
 </part>
 <part name="C2" library="microbuilder" deviceset="CAP_CERAMIC" device="0805" value="10uF/16V">
-<attribute name="MPN" value="EMK212ABJ106KG-T"/>
+<attribute name="MPN" value="LMK212BJ106KG-T"/>
 </part>
 <part name="C5" library="microbuilder" deviceset="CAP_CERAMIC" device="0805" value="1.0uF">
@@
 </part>
 <part name="C3" library="microbuilder" deviceset="CAP_CERAMIC" device="0805" value="10uF">
-<attribute name="MPN" value="EMK212ABJ106KG-T"/>
+<attribute name="MPN" value="LMK212BJ106KG-T"/>
 </part>
 <part name="GND1" library="supply1" library_urn="urn:adsk.eagle:library:371" deviceset="GND" device=""/>
@@
 </part>
 <part name="C6" library="microbuilder" deviceset="CAP_CERAMIC" device="0805" value="10uF">
-<attribute name="MPN" value="EMK212ABJ106KG-T"/>
+<attribute name="MPN" value="LMK212BJ106KG-T"/>
 </part>
 <part name="L1" library="microbuilder" deviceset="INDUCTOR" device="" value="10uH">
@@
 <part name="GND5" library="supply1" library_urn="urn:adsk.eagle:library:371" deviceset="GND" device=""/>
 <part name="C7" library="microbuilder" deviceset="CAP_CERAMIC" device="0805" value="0.1uF">
-<attribute name="MPN" value="08051C104J4T4A"/>
+<attribute name="MPN" value="C0805C104M3RACTU"/>
 </part>
 <part name="P+2" library="supply1" library_urn="urn:adsk.eagle:library:371" deviceset="+12V" device="" value="+13V"/>
@@
 </part>
 <part name="C4" library="microbuilder" deviceset="CAP_CERAMIC" device="0805" value="10uF/16V">
-<attribute name="MPN" value="EMK212ABJ106KG-T"/>
+<attribute name="MPN" value="LMK212BJ106KG-T"/>
 </part>
 <part name="D1" library="microbuilder" deviceset="DIODE" device="SOD-323" value="1N4148">
