File: pcb/usb.brd (EAGLE design)
At the start: 26.2 x 26.2 mm, 27 parts, among them J1 JSTPH, Q1 ZXMP6A13FTA, Q2 mmbt2222, Q3 mmbt2222, U1 MIC5225-3.3v, U2 CH340C, U3 MCP73831T-2ACI/OT, X1 SM02B-SRSS-TB

Commit message: changed some part numbers
Parts:
- CHG: value RED -> YELLOW
- ON: value RED -> WHITE
Changed lines of the file:
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@@
 <drawing>
 <settings>
-<setting alwaysvectorfont="yes"/>
+<setting alwaysvectorfont="no"/>
 <setting keepoldvectorfont="yes"/>
 <setting verticaltext="up"/>
@@
 <attribute name="VALUE" x="21.336" y="18.615" size="0.4064" layer="27" ratio="10" rot="R90"/>
 </element>
-<element name="CHG" library="microbuilder" package="CHIPLED_0805_NOOUTLINE" value="RED" x="19.304" y="2.54" smashed="yes" rot="MR0">
-<attribute name="MPN" value="SMLD12E3N1WT86" x="19.304" y="2.54" size="1.778" layer="28" rot="MR0" display="off"/>
+<element name="CHG" library="microbuilder" package="CHIPLED_0805_NOOUTLINE" value="YELLOW" x="19.304" y="2.54" smashed="yes" rot="MR0">
+<attribute name="MPN" value="NCD0805W2" x="19.304" y="2.54" size="1.778" layer="28" rot="MR0" display="off"/>
 <attribute name="NAME" x="20.193" y="4.572" size="0.8128" layer="26" ratio="18" rot="MR0"/>
 <attribute name="VALUE" x="17.907" y="0.762" size="0.4064" layer="28" ratio="10" rot="MR90"/>
@@
 </element>
 <element name="C1" library="adafruit" library_urn="urn:adsk.eagle:library:420" package="C0805" package3d_urn="urn:adsk.eagle:package:6240337/1" override_package3d_urn="urn:adsk.eagle:package:21520831/3" override_package_urn="urn:adsk.eagle:footprint:6239686/1" value="10µF" x="16.51" y="20.574" smashed="yes" rot="R90">
-<attribute name="MPN" value="LMK212BJ106KG-T" x="16.51" y="20.574" size="1.778" layer="27" rot="R90" display="off"/>
+<attribute name="MPN" value="CL21A106KPFNNNE" x="16.51" y="20.574" size="1.778" layer="27" rot="R90" display="off"/>
 <attribute name="NAME" x="15.621" y="22.606" size="0.8128" layer="25"/>
 <attribute name="VALUE" x="18.796" y="19.685" size="1.27" layer="27" rot="R90"/>
 </element>
 <element name="C3" library="adafruit" library_urn="urn:adsk.eagle:library:420" package="C0805" package3d_urn="urn:adsk.eagle:package:6240337/1" override_package3d_urn="urn:adsk.eagle:package:21520830/2" override_package_urn="urn:adsk.eagle:footprint:6239686/1" value="10µF" x="20.828" y="19.05" smashed="yes" rot="R180">
-<attribute name="MPN" value="LMK212BJ106KG-T" x="20.828" y="19.05" size="1.778" layer="27" rot="R180" display="off"/>
+<attribute name="MPN" value="CL21A106KPFNNNE" x="20.828" y="19.05" size="1.778" layer="27" rot="R180" display="off"/>
 <attribute name="NAME" x="21.971" y="20.193" size="0.8128" layer="25"/>
 <attribute name="VALUE" x="21.717" y="21.336" size="1.27" layer="27" rot="R180"/>
@@
 <attribute name="VALUE" value="1.0uF" x="15.748" y="4.572" size="0.4064" layer="27" font="vector"/>
 </element>
-<element name="ON" library="microbuilder" package="CHIPLED_0805_NOOUTLINE" value="RED" x="6.858" y="2.54" smashed="yes" rot="MR180">
-<attribute name="MPN" value="SMLEN3WBC8W1" x="6.858" y="2.54" size="1.778" layer="28" rot="MR180" display="off"/>
+<element name="ON" library="microbuilder" package="CHIPLED_0805_NOOUTLINE" value="WHITE" x="6.858" y="2.54" smashed="yes" rot="MR180">
+<attribute name="MPN" value="NCD0805W2" x="6.858" y="2.54" size="1.778" layer="28" rot="MR180" display="off"/>
 <attribute name="NAME" x="6.096" y="5.334" size="0.8128" layer="26" ratio="18" rot="MR180"/>
 <attribute name="VALUE" x="8.255" y="4.318" size="0.4064" layer="28" ratio="10" rot="MR270"/>
@@
 </element>
 <element name="R1" library="adafruit" library_urn="urn:adsk.eagle:library:420" package="R0805" package3d_urn="urn:adsk.eagle:package:6240566/1" override_package3d_urn="urn:adsk.eagle:package:21520834/2" override_package_urn="urn:adsk.eagle:footprint:6239920/1" value="100K" x="12.827" y="20.447" smashed="yes" rot="R270">
-<attribute name="MPN" value="CR0805AFX-1003EAS" x="12.827" y="20.447" size="1.778" layer="27" rot="R270" display="off"/>
+<attribute name="MPN" value="0805W8F1003T5E" x="12.827" y="20.447" size="1.778" layer="27" rot="R270" display="off"/>
 <attribute name="NAME" x="11.811" y="22.479" size="0.8128" layer="25"/>
 <attribute name="VALUE" x="10.541" y="21.209" size="1.27" layer="27" rot="R270"/>
 </element>
 <element name="C2" library="adafruit" library_urn="urn:adsk.eagle:library:420" package="C0805" package3d_urn="urn:adsk.eagle:package:6240337/1" override_package3d_urn="urn:adsk.eagle:package:21520809/2" override_package_urn="urn:adsk.eagle:footprint:6239686/1" value="10uF" x="8.001" y="16.002" smashed="yes">
-<attribute name="MPN" value="LMK212BJ106KG-T" x="8.001" y="16.002" size="1.778" layer="27" display="off"/>
+<attribute name="MPN" value="CL21A106KPFNNNE" x="8.001" y="16.002" size="1.778" layer="27" display="off"/>
 <attribute name="NAME" x="8.128" y="17.018" size="0.8128" layer="25"/>
 <attribute name="VALUE" x="7.112" y="13.716" size="1.27" layer="27"/>
