File: pcb/usb.sch (EAGLE design)
At the start: 26 parts, among them J1 JSTPH, Q1 ZXMP6A13FTA, Q2 mmbt2222, Q3 mmbt2222, U1 MIC5225-3.3v, U2 CH340C, U3 MCP73831T-2ACI/OT, X1 SM02B-SRSS-TB

Commit message: added thru-hole prop to usb board
Parts:
- J2, JP1, JP2: THRU-HOLE (none) -> 1
Changed lines of the file:
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@@
 <?xml version="1.0" encoding="utf-8"?>
 <!DOCTYPE eagle SYSTEM "eagle.dtd">
-<eagle version="9.6.2">
+<eagle version="9.5.0">
 <drawing>
 <settings>
@@
 <part name="JP2" library="adafruit" library_urn="urn:adsk.eagle:library:420" deviceset="PINHD-1X8" device="CLEANBIG" package3d_urn="urn:adsk.eagle:package:6240708/1" override_package3d_urn="urn:adsk.eagle:package:21520758/2" override_package_urn="urn:adsk.eagle:footprint:6240062/1">
 <attribute name="MPN" value="8Fx1L-254mm"/>
+<attribute name="THRU-HOLE" value="1"/>
 </part>
 <part name="JP1" library="adafruit" library_urn="urn:adsk.eagle:library:420" deviceset="PINHD-1X8" device="CLEANBIG" package3d_urn="urn:adsk.eagle:package:6240708/1" override_package3d_urn="urn:adsk.eagle:package:21520677/2" override_package_urn="urn:adsk.eagle:footprint:6240062/1">
 <attribute name="MPN" value="8Fx1L-254mm"/>
+<attribute name="THRU-HOLE" value="1"/>
 </part>
 <part name="J2" library="Wurth_Elektronik_Electromechanic_Input-Output_Connectors_rev19b_wider_slots" deviceset="614105150621" device="" package3d_urn="urn:adsk.eagle:package:3360156/4" override_package3d_urn="urn:adsk.eagle:package:21520771/2" override_package_urn="urn:adsk.eagle:footprint:21520772/1">
 <attribute name="MPN" value="614105150621"/>
+<attribute name="THRU-HOLE" value="1"/>
 </part>
 <part name="D1" library="microbuilder" deviceset="DIODE-SCHOTTKY" device="SOD-123" override_package3d_urn="urn:adsk.eagle:package:21520835/2" override_package_urn="urn:adsk.eagle:footprint:21520836/1" value="MBR120">
@@
 <attribute name="VALUE" x="64.77" y="35.56" size="1.778" layer="96" rot="R180"/>
 <attribute name="MPN" x="58.42" y="20.32" size="1.778" layer="96" rot="R180" display="off"/>
+<attribute name="THRU-HOLE" x="58.42" y="20.32" size="1.778" layer="96" rot="R180" display="off"/>
 </instance>
 <instance part="JP1" gate="G$1" x="48.26" y="22.86" smashed="yes">
@@
 <attribute name="VALUE" x="41.91" y="7.62" size="1.778" layer="96"/>
 <attribute name="MPN" x="48.26" y="22.86" size="1.778" layer="96" display="off"/>
+<attribute name="THRU-HOLE" x="48.26" y="22.86" size="1.778" layer="96" display="off"/>
 </instance>
 <instance part="J2" gate="G$1" x="182.88" y="22.86" smashed="yes">
@@
 <attribute name="VALUE" x="180.34" y="8.89" size="1.778" layer="96"/>
 <attribute name="MPN" x="182.88" y="22.86" size="1.778" layer="96" display="off"/>
+<attribute name="THRU-HOLE" x="182.88" y="22.86" size="1.778" layer="96" display="off"/>
 </instance>
 <instance part="D1" gate="G$1" x="25.4" y="68.58" smashed="yes">

Commit message: added bottom prop to usb connector
Parts:
- J2: BOTTOM (none) -> 1
Changed lines of the file:
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@@
 </part>
 <part name="J2" library="Wurth_Elektronik_Electromechanic_Input-Output_Connectors_rev19b_wider_slots" deviceset="614105150621" device="" package3d_urn="urn:adsk.eagle:package:3360156/4" override_package3d_urn="urn:adsk.eagle:package:21520771/2" override_package_urn="urn:adsk.eagle:footprint:21520772/1">
+<attribute name="BOTTOM" value="1"/>
 <attribute name="MPN" value="614105150621"/>
 <attribute name="THRU-HOLE" value="1"/>
@@
 <attribute name="MPN" x="182.88" y="22.86" size="1.778" layer="96" display="off"/>
 <attribute name="THRU-HOLE" x="182.88" y="22.86" size="1.778" layer="96" display="off"/>
+<attribute name="BOTTOM" x="182.88" y="22.86" size="1.778" layer="96" display="off"/>
 </instance>
 <instance part="D1" gate="G$1" x="25.4" y="68.58" smashed="yes">

Commit message: added populate attr
Parts:
- J1: POPULATE (none) -> 0
- R3: value 10K\ -> 10K
Changed lines of the file:
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@@
 <attribute name="MPN" value="ESR10EZPJ102"/>
 </part>
-<part name="J1" library="SparkFun-Connectors" library_urn="urn:adsk.eagle:library:513" deviceset="CONN_02" device="" package3d_urn="urn:adsk.eagle:package:38039/1" value="JSTPH"/>
+<part name="J1" library="SparkFun-Connectors" library_urn="urn:adsk.eagle:library:513" deviceset="CONN_02" device="" package3d_urn="urn:adsk.eagle:package:38039/1" value="JSTPH">
+<attribute name="POPULATE" value="0"/>
+</part>
 <part name="C1" library="adafruit" library_urn="urn:adsk.eagle:library:420" deviceset="C-US" device="C0805" package3d_urn="urn:adsk.eagle:package:6240337/1" override_package3d_urn="urn:adsk.eagle:package:21520831/3" override_package_urn="urn:adsk.eagle:footprint:6239686/1" value="10µF">
 <attribute name="MPN" value="LMK212BJ106KG-T"/>
@@
 <attribute name="MPN" value="LMK212BJ106KG-T"/>
 </part>
-<part name="R3" library="adafruit" library_urn="urn:adsk.eagle:library:420" deviceset="R-US_" device="R0805" package3d_urn="urn:adsk.eagle:package:6240566/1" override_package3d_urn="urn:adsk.eagle:package:21520802/2" override_package_urn="urn:adsk.eagle:footprint:6239920/1" value="10K\">
+<part name="R3" library="adafruit" library_urn="urn:adsk.eagle:library:420" deviceset="R-US_" device="R0805" package3d_urn="urn:adsk.eagle:package:6240566/1" override_package3d_urn="urn:adsk.eagle:package:21520802/2" override_package_urn="urn:adsk.eagle:footprint:6239920/1" value="10K">
 <attribute name="MPN" value="CRCW080510K0FKEAC"/>
 </part>
@@
 <attribute name="VALUE" x="119.38" y="126.746" size="1.778" layer="96" font="vector" rot="R180"/>
 <attribute name="NAME" x="119.38" y="116.332" size="1.778" layer="95" font="vector" rot="R180"/>
+<attribute name="POPULATE" x="116.84" y="121.92" size="1.778" layer="96" rot="R180" display="off"/>
 </instance>
 <instance part="C1" gate="G$1" x="17.78" y="111.76" smashed="yes">

Commit message: changed some part numbers
Parts:
- C1, C2, C3: MPN LMK212BJ106KG-T -> CL21A106KPFNNNE
- CHG: value RED -> YELLOW; MPN SMLD12E3N1WT86 -> NCD0805W2
- ON: value RED -> WHITE; MPN SMLEN3WBC8W1 -> NCD0805W2
- R1: MPN CR0805AFX-1003EAS -> 0805W8F1003T5E
Changed lines of the file:
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@@
 <attribute name="MPN" value="MCP73831T-2ACI/OT"/>
 </part>
-<part name="CHG" library="microbuilder" deviceset="LED" device="0805_NOOUTLINE" value="RED">
-<attribute name="MPN" value="SMLD12E3N1WT86"/>
+<part name="CHG" library="microbuilder" deviceset="LED" device="0805_NOOUTLINE" value="YELLOW">
+<attribute name="MPN" value="NCD0805W2"/>
 </part>
 <part name="R2" library="adafruit" library_urn="urn:adsk.eagle:library:420" deviceset="R-US_" device="R0805" package3d_urn="urn:adsk.eagle:package:6240566/1" override_package3d_urn="urn:adsk.eagle:package:21520789/2" override_package_urn="urn:adsk.eagle:footprint:6239920/1" value="1K">
@@
 </part>
 <part name="C1" library="adafruit" library_urn="urn:adsk.eagle:library:420" deviceset="C-US" device="C0805" package3d_urn="urn:adsk.eagle:package:6240337/1" override_package3d_urn="urn:adsk.eagle:package:21520831/3" override_package_urn="urn:adsk.eagle:footprint:6239686/1" value="10µF">
-<attribute name="MPN" value="LMK212BJ106KG-T"/>
+<attribute name="MPN" value="CL21A106KPFNNNE"/>
 </part>
 <part name="C3" library="adafruit" library_urn="urn:adsk.eagle:library:420" deviceset="C-US" device="C0805" package3d_urn="urn:adsk.eagle:package:6240337/1" override_package3d_urn="urn:adsk.eagle:package:21520830/2" override_package_urn="urn:adsk.eagle:footprint:6239686/1" value="10µF">
-<attribute name="MPN" value="LMK212BJ106KG-T"/>
+<attribute name="MPN" value="CL21A106KPFNNNE"/>
 </part>
 <part name="R3" library="adafruit" library_urn="urn:adsk.eagle:library:420" deviceset="R-US_" device="R0805" package3d_urn="urn:adsk.eagle:package:6240566/1" override_package3d_urn="urn:adsk.eagle:package:21520802/2" override_package_urn="urn:adsk.eagle:footprint:6239920/1" value="10K">
@@
 <attribute name="MPN" value="C0805C104M3RACTU"/>
 </part>
-<part name="ON" library="microbuilder" deviceset="LED" device="0805_NOOUTLINE" value="RED">
-<attribute name="MPN" value="SMLEN3WBC8W1"/>
+<part name="ON" library="microbuilder" deviceset="LED" device="0805_NOOUTLINE" value="WHITE">
+<attribute name="MPN" value="NCD0805W2"/>
 </part>
 <part name="R4" library="adafruit" library_urn="urn:adsk.eagle:library:420" deviceset="R-US_" device="R0805" package3d_urn="urn:adsk.eagle:package:6240566/1" override_package3d_urn="urn:adsk.eagle:package:21520793/2" override_package_urn="urn:adsk.eagle:footprint:6239920/1" value="1K">
@@
 </part>
 <part name="R1" library="adafruit" library_urn="urn:adsk.eagle:library:420" deviceset="R-US_" device="R0805" package3d_urn="urn:adsk.eagle:package:6240566/1" override_package3d_urn="urn:adsk.eagle:package:21520834/2" override_package_urn="urn:adsk.eagle:footprint:6239920/1" value="100K">
-<attribute name="MPN" value="CR0805AFX-1003EAS"/>
+<attribute name="MPN" value="0805W8F1003T5E"/>
 </part>
 <part name="SUPPLY8" library="SparkFun-PowerSymbols" deviceset="3.3V" device=""/>
@@
 <part name="GND11" library="SparkFun-PowerSymbols" library_urn="urn:adsk.eagle:library:530" deviceset="GND" device=""/>
 <part name="C2" library="adafruit" library_urn="urn:adsk.eagle:library:420" deviceset="C-US" device="C0805" package3d_urn="urn:adsk.eagle:package:6240337/1" override_package3d_urn="urn:adsk.eagle:package:21520809/2" override_package_urn="urn:adsk.eagle:footprint:6239686/1" value="10uF">
-<attribute name="MPN" value="LMK212BJ106KG-T"/>
+<attribute name="MPN" value="CL21A106KPFNNNE"/>
 </part>
 <part name="X1" library="con-jst2.rpt" deviceset="?M02B-SRSS-TB" device="S" override_package3d_urn="urn:adsk.eagle:package:21520875/2" override_package_urn="urn:adsk.eagle:footprint:21520876/1"/>

Commit message: replaced 0805 10k with 0603
Parts:
- R5, R6: MPN CRCW080510K0FKEAC -> RC0603FR-0710KL
Changed lines of the file:
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@@
 </part>
 <part name="R6" library="adafruit" library_urn="urn:adsk.eagle:library:420" deviceset="R-US_" device="R0603" package3d_urn="urn:adsk.eagle:package:6240565/1" override_package3d_urn="urn:adsk.eagle:package:21520799/2" override_package_urn="urn:adsk.eagle:footprint:6239919/1" value="10K">
-<attribute name="MPN" value="CRCW080510K0FKEAC"/>
+<attribute name="MPN" value="RC0603FR-0710KL"/>
 </part>
 <part name="R5" library="adafruit" library_urn="urn:adsk.eagle:library:420" deviceset="R-US_" device="R0603" package3d_urn="urn:adsk.eagle:package:6240565/1" override_package3d_urn="urn:adsk.eagle:package:21520797/2" override_package_urn="urn:adsk.eagle:footprint:6239919/1" value="10K">
-<attribute name="MPN" value="CRCW080510K0FKEAC"/>
+<attribute name="MPN" value="RC0603FR-0710KL"/>
 </part>
 <part name="Q3" library="SparkFun" deviceset="TRANSISTOR_NPN" device="SOT23-3" value="mmbt2222">

Commit message: added MPN for jst connector
Parts:
- X1: MPN (none) -> SM02B-SRSS-TB
Changed lines of the file:
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@@
 <attribute name="MPN" value="CL21A106KPFNNNE"/>
 </part>
-<part name="X1" library="con-jst2.rpt" deviceset="?M02B-SRSS-TB" device="S" override_package3d_urn="urn:adsk.eagle:package:21520875/2" override_package_urn="urn:adsk.eagle:footprint:21520876/1"/>
+<part name="X1" library="con-jst2.rpt" deviceset="?M02B-SRSS-TB" device="S" override_package3d_urn="urn:adsk.eagle:package:21520875/2" override_package_urn="urn:adsk.eagle:footprint:21520876/1">
+<attribute name="MPN" value="SM02B-SRSS-TB"/>
+</part>
 <part name="SUPPLY9" library="SparkFun-PowerSymbols" library_urn="urn:adsk.eagle:library:530" deviceset="V_BATT" device=""/>
 <part name="GND12" library="SparkFun-PowerSymbols" library_urn="urn:adsk.eagle:library:530" deviceset="GND" device=""/>
@@
 <attribute name="NAME" x="132.08" y="121.158" size="1.524" layer="95"/>
 <attribute name="VALUE" x="128.778" y="123.317" size="1.524" layer="96"/>
+<attribute name="MPN" x="129.54" y="121.92" size="1.778" layer="96" display="off"/>
 </instance>
 <instance part="X1" gate="-2" x="129.54" y="119.38" smashed="yes">

Commit message: updated part number for usb connector
Parts:
- J2: MPN 614105150621 -> U-D-M5DD-W-1
Changed lines of the file:
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@@
 <part name="J2" library="Wurth_Elektronik_Electromechanic_Input-Output_Connectors_rev19b_wider_slots" deviceset="614105150621" device="" package3d_urn="urn:adsk.eagle:package:3360156/4" override_package3d_urn="urn:adsk.eagle:package:21520771/2" override_package_urn="urn:adsk.eagle:footprint:21520772/1">
 <attribute name="BOTTOM" value="1"/>
-<attribute name="MPN" value="614105150621"/>
+<attribute name="MPN" value="U-D-M5DD-W-1"/>
 <attribute name="THRU-HOLE" value="1"/>
 </part>
