File: pcb/microcontroller.sch (EAGLE design)
At the start: 14 parts, among them J1 SMD, U1 MMA8452Q

Commit message: change populate field for some parts
Parts:
- C3, C4, U1: POPULATE 0 -> 1
Changed lines of the file:
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@@
 <?xml version="1.0" encoding="utf-8"?>
 <!DOCTYPE eagle SYSTEM "eagle.dtd">
-<eagle version="9.6.2">
+<eagle version="9.5.0">
 <drawing>
 <settings>
@@
 <part name="U1" library="SparkX" deviceset="MMA8452Q" device="" override_package3d_urn="urn:adsk.eagle:package:21520916/2" override_package_urn="urn:adsk.eagle:footprint:21520917/1">
 <attribute name="MPN" value="MMA8452QR1"/>
-<attribute name="POPULATE" value="0"/>
+<attribute name="POPULATE" value="1"/>
 </part>
 <part name="LED1" library="adafruit" library_urn="urn:adsk.eagle:library:420" deviceset="WS2812B" device="5050" package3d_urn="urn:adsk.eagle:package:6240942/1">
@@
 <part name="C4" library="adafruit" library_urn="urn:adsk.eagle:library:420" deviceset="C-US" device="C0805" package3d_urn="urn:adsk.eagle:package:6240337/1" override_package3d_urn="urn:adsk.eagle:package:21520929/2" override_package_urn="urn:adsk.eagle:footprint:6239686/1" value=".1uF">
 <attribute name="MPN" value="C0805C104M3RACTU"/>
-<attribute name="POPULATE" value="0"/>
+<attribute name="POPULATE" value="1"/>
 </part>
 <part name="C3" library="adafruit" library_urn="urn:adsk.eagle:library:420" deviceset="C-US" device="C0805" package3d_urn="urn:adsk.eagle:package:6240337/1" override_package3d_urn="urn:adsk.eagle:package:21520930/2" override_package_urn="urn:adsk.eagle:footprint:6239686/1" value="10uF">
 <attribute name="MPN" value="LMK212BJ106KG-T"/>
-<attribute name="POPULATE" value="0"/>
+<attribute name="POPULATE" value="1"/>
 </part>
 <part name="SUPPLY1" library="SparkFun-PowerSymbols" deviceset="3.3V" device=""/>

Commit message: added thru-hole parameters and updated eagle export script
Parts:
- JP1, JP2: BOTTOM (none) -> 1; THRU-HOLE (none) -> 1
Changed lines of the file:
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@@
 </part>
 <part name="JP2" library="adafruit" library_urn="urn:adsk.eagle:library:420" deviceset="PINHD-1X8" device="CLEANBIG" package3d_urn="urn:adsk.eagle:package:6240708/1" override_package3d_urn="urn:adsk.eagle:package:21520910/2" override_package_urn="urn:adsk.eagle:footprint:6240062/1">
+<attribute name="BOTTOM" value="1"/>
 <attribute name="MPN" value="8Fx1L-254mm"/>
+<attribute name="THRU-HOLE" value="1"/>
 </part>
 <part name="JP1" library="adafruit" library_urn="urn:adsk.eagle:library:420" deviceset="PINHD-1X8" device="CLEANBIG" package3d_urn="urn:adsk.eagle:package:6240708/1" override_package3d_urn="urn:adsk.eagle:package:21520912/2" override_package_urn="urn:adsk.eagle:footprint:6240062/1">
+<attribute name="BOTTOM" value="1"/>
 <attribute name="MPN" value="8Fx1L-254mm"/>
+<attribute name="THRU-HOLE" value="1"/>
 </part>
 <part name="GND6" library="SparkFun" deviceset="GND" device=""/>
@@
 <attribute name="VALUE" x="153.67" y="20.32" size="1.778" layer="96" rot="R180"/>
 <attribute name="MPN" x="147.32" y="5.08" size="1.778" layer="96" rot="R180" display="off"/>
+<attribute name="THRU-HOLE" x="147.32" y="5.08" size="1.778" layer="96" rot="R180" display="off"/>
+<attribute name="BOTTOM" x="147.32" y="5.08" size="1.778" layer="96" rot="R180" display="off"/>
 </instance>
 <instance part="JP1" gate="G$1" x="137.16" y="7.62" smashed="yes">
@@
 <attribute name="VALUE" x="130.81" y="-7.62" size="1.778" layer="96"/>
 <attribute name="MPN" x="137.16" y="7.62" size="1.778" layer="96" display="off"/>
+<attribute name="THRU-HOLE" x="137.16" y="7.62" size="1.778" layer="96" display="off"/>
+<attribute name="BOTTOM" x="137.16" y="7.62" size="1.778" layer="96" display="off"/>
 </instance>
 <instance part="GND6" gate="1" x="251.46" y="63.5" smashed="yes">

Commit message: updated part numbers
Parts:
- JP1, JP2: MPN 8Fx1L-254mm -> 83-15410
- X1: MPN ESP12 -> ESP-12F(ESP8266MOD)
Changed lines of the file:
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@@
 </part>
 <part name="X1" library="adafruit" library_urn="urn:adsk.eagle:library:420" deviceset="ESP-12" device="">
-<attribute name="MPN" value="ESP12"/>
+<attribute name="MPN" value="ESP-12F(ESP8266MOD)"/>
 </part>
 <part name="JP2" library="adafruit" library_urn="urn:adsk.eagle:library:420" deviceset="PINHD-1X8" device="CLEANBIG" package3d_urn="urn:adsk.eagle:package:6240708/1" override_package3d_urn="urn:adsk.eagle:package:21520910/2" override_package_urn="urn:adsk.eagle:footprint:6240062/1">
 <attribute name="BOTTOM" value="1"/>
-<attribute name="MPN" value="8Fx1L-254mm"/>
+<attribute name="MPN" value="83-15410"/>
 <attribute name="THRU-HOLE" value="1"/>
 </part>
 <part name="JP1" library="adafruit" library_urn="urn:adsk.eagle:library:420" deviceset="PINHD-1X8" device="CLEANBIG" package3d_urn="urn:adsk.eagle:package:6240708/1" override_package3d_urn="urn:adsk.eagle:package:21520912/2" override_package_urn="urn:adsk.eagle:footprint:6240062/1">
 <attribute name="BOTTOM" value="1"/>
-<attribute name="MPN" value="8Fx1L-254mm"/>
+<attribute name="MPN" value="83-15410"/>
 <attribute name="THRU-HOLE" value="1"/>
 </part>
