File: pcb/oled.brd (EAGLE design)
At the start: 26.2 x 26.2 mm, 21 parts, among them U1 UG-2828GDEDF11, U2 FAN5331SX

Commit message: Revert OLED board to use 3.3V for input to the 13V FAN5331 boost
Connections:
- net +3V3: now also C6.1, L1.P$1, U2.4, U2.5
- net VIN: no longer C6.1, L1.P$1, U2.4, U2.5
Routing:
- net VIN: track 25.2 -> 0.00 mm
- net +3V3: track 37.9 -> 53.8 mm
Other:
- board text added: "BWS OLED V4"
- board text removed: "BWS OLED V3"
Changed lines of the file:
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@@
 <?xml version="1.0" encoding="utf-8"?>
 <!DOCTYPE eagle SYSTEM "eagle.dtd">
-<eagle version="9.5.0">
+<eagle version="9.6.2">
 <drawing>
 <settings>
-<setting alwaysvectorfont="yes"/>
+<setting alwaysvectorfont="no"/>
 <setting keepoldvectorfont="yes"/>
 <setting verticaltext="up"/>
@@
 </layers>
 <board>
-<fusionsync huburn="a.cGVyc29uYWw6dWUyODFhMTI5" projecturn="a.cGVyc29uYWw6dWUyODFhMTI5IzIwMTkwOTE3MjE1ODk1MzI2" f3durn="urn:adsk.wipprod:dm.lineage:P5lhZWs8S_KHtQ88bDf2NQ" pcbguid="d3e705c3-1af4-4cef-b1e2-384e1dcb5e4e" lastpulledtime="" lastsyncedchangeguid="5ba198aa-53f5-64b5-e4eb-32003e20bcfd"/>
+<fusionsync huburn="a.cGVyc29uYWw6dWUyODFhMTI5" projecturn="a.cGVyc29uYWw6dWUyODFhMTI5IzIwMTkwOTE3MjE1ODk1MzI2" f3durn="urn:adsk.wipprod:dm.lineage:P5lhZWs8S_KHtQ88bDf2NQ" pcbguid="d3e705c3-1af4-4cef-b1e2-384e1dcb5e4e" lastpulledtime="" lastsyncedchangeguid="5ba198aa-53f5-64b5-e4eb-32003e20bcfd" latestrevisionid="" lastsyncedrevisionid="" lastboardhashguid="" lastpushedtime="" linktopcb3d="false"/>
 <plain>
 <wire x1="0" y1="26.162" x2="0" y2="0" width="0" layer="20" grouprefs="EVERYTHING"/>
@@
 <text x="2.794" y="4.572" size="0.8128" layer="26" rot="MR180" grouprefs="EVERYTHING">VIN</text>
 <text x="16.637" y="22.606" size="0.8128" layer="25" font="vector">BWS
-OLED V3</text>
+OLED V4</text>
 </plain>
 <attributes>
@@
 <via x="17.3736" y="8.4328" extent="1-16" drill="0.4"/>
 <via x="14.224" y="5.588" extent="1-16" drill="0.4"/>
+<contactref element="C6" pad="1"/>
+<contactref element="U2" pad="5"/>
+<contactref element="U2" pad="4"/>
+<contactref element="L1" pad="P$1"/>
+<wire x1="12.2936" y1="18.4912" x2="10.4648" y2="18.4912" width="0.4064" layer="1"/>
+<wire x1="10.4648" y1="18.4912" x2="10.43" y2="18.5119" width="0.4064" layer="1"/>
+<wire x1="12.2936" y1="18.4912" x2="12.33" y2="18.5119" width="0.4064" layer="1"/>
+<wire x1="10.4648" y1="16.9672" x2="10.4648" y2="15.4432" width="0.4064" layer="1"/>
+<wire x1="10.2616" y1="17.1704" x2="10.4648" y2="16.9672" width="0.4064" layer="1"/>
+<wire x1="10.2616" y1="17.78" x2="10.2616" y2="17.1704" width="0.4064" layer="1"/>
+<wire x1="10.4648" y1="17.9832" x2="10.2616" y2="17.78" width="0.4064" layer="1"/>
+<wire x1="10.4648" y1="18.288" x2="10.4648" y2="17.9832" width="0.4064" layer="1"/>
+<wire x1="10.4648" y1="15.4432" x2="10.483" y2="15.367" width="0.4064" layer="1"/>
+<wire x1="10.4648" y1="18.288" x2="10.43" y2="18.5119" width="0.4064" layer="1"/>
+<wire x1="13.208" y1="18.6944" x2="15.1384" y2="18.6944" width="0.4064" layer="1"/>
+<wire x1="13.1064" y1="18.5928" x2="13.208" y2="18.6944" width="0.4064" layer="1"/>
+<wire x1="12.4968" y1="18.5928" x2="13.1064" y2="18.5928" width="0.4064" layer="1"/>
+<wire x1="15.1384" y1="18.6944" x2="15.19" y2="18.685" width="0.4064" layer="1"/>
+<wire x1="12.4968" y1="18.5928" x2="12.33" y2="18.5119" width="0.4064" layer="1"/>
+<wire x1="6.7633375" y1="10.4346" x2="7.1284" y2="10.7996625" width="0.4064" layer="1"/>
+<wire x1="7.1284" y1="10.7996625" x2="7.1284" y2="12.1068" width="0.4064" layer="1"/>
+<wire x1="7.1284" y1="12.1068" x2="10.4648" y2="15.4432" width="0.4064" layer="1"/>
+<wire x1="5.845" y1="9.591" x2="6.6886" y2="10.4346" width="0.4064" layer="1"/>
+<wire x1="6.6886" y1="10.4346" x2="6.7633375" y2="10.4346" width="0.4064" layer="1"/>
 </signal>
 <signal name="D1/GPIO5">
@@
 </signal>
 <signal name="VIN" class="1">
-<contactref element="C6" pad="1"/>
-<contactref element="U2" pad="5"/>
-<contactref element="U2" pad="4"/>
-<contactref element="L1" pad="P$1"/>
 <contactref element="JP1" pad="8"/>
-<wire x1="12.2936" y1="18.4912" x2="10.4648" y2="18.4912" width="0.4064" layer="1"/>
-<wire x1="10.4648" y1="18.4912" x2="10.43" y2="18.5119" width="0.4064" layer="1"/>
-<wire x1="12.2936" y1="18.4912" x2="12.33" y2="18.5119" width="0.4064" layer="1"/>
-<wire x1="10.4648" y1="16.9672" x2="10.4648" y2="15.4432" width="0.4064" layer="1"/>
-<wire x1="10.2616" y1="17.1704" x2="10.4648" y2="16.9672" width="0.4064" layer="1"/>
-<wire x1="10.2616" y1="17.78" x2="10.2616" y2="17.1704" width="0.4064" layer="1"/>
-<wire x1="10.4648" y1="17.9832" x2="10.2616" y2="17.78" width="0.4064" layer="1"/>
-<wire x1="10.4648" y1="18.288" x2="10.4648" y2="17.9832" width="0.4064" layer="1"/>
-<wire x1="10.4648" y1="15.4432" x2="10.483" y2="15.367" width="0.4064" layer="1"/>
-<wire x1="10.4648" y1="18.288" x2="10.43" y2="18.5119" width="0.4064" layer="1"/>
-<wire x1="13.208" y1="18.6944" x2="15.1384" y2="18.6944" width="0.4064" layer="1"/>
-<wire x1="13.1064" y1="18.5928" x2="13.208" y2="18.6944" width="0.4064" layer="1"/>
-<wire x1="12.4968" y1="18.5928" x2="13.1064" y2="18.5928" width="0.4064" layer="1"/>
-<wire x1="15.1384" y1="18.6944" x2="15.19" y2="18.685" width="0.4064" layer="1"/>
-<wire x1="12.4968" y1="18.5928" x2="12.33" y2="18.5119" width="0.4064" layer="1"/>
-<wire x1="1.9304" y1="4.2672" x2="1.7272" y2="4.2672" width="0.4064" layer="1"/>
-<wire x1="3.9624" y1="6.2992" x2="1.9304" y2="4.2672" width="0.4064" layer="1"/>
-<wire x1="3.9624" y1="12.4968" x2="3.9624" y2="6.2992" width="0.4064" layer="1"/>
-<wire x1="6.604" y1="15.1384" x2="3.9624" y2="12.4968" width="0.4064" layer="1"/>
-<wire x1="10.2616" y1="15.1384" x2="6.604" y2="15.1384" width="0.4064" layer="1"/>
-<wire x1="10.3632" y1="15.24" x2="10.2616" y2="15.1384" width="0.4064" layer="1"/>
-<wire x1="1.7272" y1="4.2672" x2="1.651" y2="4.191" width="0.4064" layer="1"/>
-<wire x1="10.3632" y1="15.24" x2="10.483" y2="15.367" width="0.4064" layer="1"/>
 </signal>
 <signal name="D6/GPIO12/MISO">

Commit message: changed 590k resistor to 620k
Parts:
- R2: value 600K -> 620K
Changed lines of the file:
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@@
 <?xml version="1.0" encoding="utf-8"?>
 <!DOCTYPE eagle SYSTEM "eagle.dtd">
-<eagle version="9.6.2">
+<eagle version="9.5.0">
 <drawing>
 <settings>
@@
 </layers>
 <board>
-<fusionsync huburn="a.cGVyc29uYWw6dWUyODFhMTI5" projecturn="a.cGVyc29uYWw6dWUyODFhMTI5IzIwMTkwOTE3MjE1ODk1MzI2" f3durn="urn:adsk.wipprod:dm.lineage:P5lhZWs8S_KHtQ88bDf2NQ" pcbguid="d3e705c3-1af4-4cef-b1e2-384e1dcb5e4e" lastpulledtime="" lastsyncedchangeguid="5ba198aa-53f5-64b5-e4eb-32003e20bcfd" latestrevisionid="" lastsyncedrevisionid="" lastboardhashguid="" lastpushedtime="" linktopcb3d="false"/>
+<fusionsync huburn="a.cGVyc29uYWw6dWUyODFhMTI5" projecturn="a.cGVyc29uYWw6dWUyODFhMTI5IzIwMTkwOTE3MjE1ODk1MzI2" f3durn="urn:adsk.wipprod:dm.lineage:P5lhZWs8S_KHtQ88bDf2NQ" pcbguid="d3e705c3-1af4-4cef-b1e2-384e1dcb5e4e" lastpulledtime="" lastsyncedchangeguid="5ba198aa-53f5-64b5-e4eb-32003e20bcfd"/>
 <plain>
 <wire x1="0" y1="26.162" x2="0" y2="0" width="0" layer="20" grouprefs="EVERYTHING"/>
@@
 </groups>
 <elements>
-<element name="R2" library="adafruit" library_urn="urn:adsk.eagle:library:420" package="R0805" package3d_urn="urn:adsk.eagle:package:6240566/1" override_package3d_urn="urn:adsk.eagle:package:21520237/2" override_package_urn="urn:adsk.eagle:footprint:6239920/1" value="600K" x="11.08" y="10.541" smashed="yes" rot="R270" grouprefs="EVERYTHING">
-<attribute name="MPN" value="ERJ-6ENF5903V" x="11.08" y="10.541" size="1.778" layer="27" rot="R270" display="off"/>
+<element name="R2" library="adafruit" library_urn="urn:adsk.eagle:library:420" package="R0805" package3d_urn="urn:adsk.eagle:package:6240566/1" override_package3d_urn="urn:adsk.eagle:package:21520237/2" override_package_urn="urn:adsk.eagle:footprint:6239920/1" value="620K" x="11.08" y="10.541" smashed="yes" rot="R270" grouprefs="EVERYTHING">
+<attribute name="MPN" value="0805W8F6203T5E" x="11.08" y="10.541" size="1.778" layer="27" rot="R270" display="off"/>
 <attribute name="NAME" x="10.287" y="12.731" size="0.8128" layer="25" font="vector"/>
 <attribute name="VALUE" x="11.018" y="12.827" size="1.016" layer="27" rot="R90"/>
