File: cad/pcb/usb.brd (EAGLE design)
At the start: 26.2 x 26.2 mm, 26 parts, among them Q1 ZXMP6A13FTA, Q2 mmbt2222, Q3 mmbt2222, U1 MIC5225-3.3v, U2 CH340C, U3 MCP73831T-2ACI/OT, X1 SM02B-SRSS-TB

Commit message: updated R2 and R4 values, changed 3.3v regulator to AP2112K-3.3
Parts:
- R2, R4: value 1K -> 5K
- U1: value MIC5225-3.3v -> AP211K-3.3
Changed lines of the file:
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@@
 </autorouter>
 <elements>
-<element name="U1" library="microbuilder" package="SOT23-5" value="MIC5225-3.3v" x="5.588" y="19.047" smashed="yes" rot="R90">
-<attribute name="MPN" value="MIC5225-3.3YM5-TR" x="5.588" y="19.047" size="1.778" layer="27" rot="R90" display="off"/>
+<element name="U1" library="microbuilder" package="SOT23-5" value="AP211K-3.3" x="5.588" y="19.047" smashed="yes" rot="R90">
+<attribute name="MPN" value="AP2112K-3.3" x="5.588" y="19.047" size="1.778" layer="27" rot="R90" display="off"/>
 <attribute name="NAME" x="5.21" y="16.764" size="0.8128" layer="25" rot="R180"/>
 <attribute name="VALUE" x="1.193" y="20.828" size="1.016" layer="27"/>
@@
 <attribute name="VALUE" x="17.907" y="0.762" size="0.4064" layer="28" ratio="10" rot="MR90"/>
 </element>
-<element name="R2" library="adafruit" library_urn="urn:adsk.eagle:library:420" package="R0805" package3d_urn="urn:adsk.eagle:package:6240566/1" override_package3d_urn="urn:adsk.eagle:package:21520789/2" override_package_urn="urn:adsk.eagle:footprint:6239920/1" value="1K" x="19.304" y="2.54" smashed="yes" rot="R270">
-<attribute name="MPN" value="ESR10EZPJ102" x="19.304" y="2.54" size="1.778" layer="27" rot="R270" display="off"/>
+<element name="R2" library="adafruit" library_urn="urn:adsk.eagle:library:420" package="R0805" package3d_urn="urn:adsk.eagle:package:6240566/1" override_package3d_urn="urn:adsk.eagle:package:21520789/2" override_package_urn="urn:adsk.eagle:footprint:6239920/1" value="5K" x="19.304" y="2.54" smashed="yes" rot="R270">
+<attribute name="MPN" value="0805W8F4871T5E" x="19.304" y="2.54" size="1.778" layer="27" rot="R270" display="off"/>
 <attribute name="NAME" x="20.701" y="0.762" size="0.8128" layer="25"/>
 <attribute name="VALUE" x="17.018" y="3.302" size="1.27" layer="27" rot="R270"/>
@@
 <attribute name="VALUE" x="8.255" y="4.318" size="0.4064" layer="28" ratio="10" rot="MR270"/>
 </element>
-<element name="R4" library="adafruit" library_urn="urn:adsk.eagle:library:420" package="R0805" package3d_urn="urn:adsk.eagle:package:6240566/1" override_package3d_urn="urn:adsk.eagle:package:21520793/2" override_package_urn="urn:adsk.eagle:footprint:6239920/1" value="1K" x="6.858" y="2.556" smashed="yes" rot="R90">
-<attribute name="MPN" value="ESR10EZPJ102" x="6.858" y="2.556" size="1.778" layer="27" rot="R90" display="off"/>
+<element name="R4" library="adafruit" library_urn="urn:adsk.eagle:library:420" package="R0805" package3d_urn="urn:adsk.eagle:package:6240566/1" override_package3d_urn="urn:adsk.eagle:package:21520793/2" override_package_urn="urn:adsk.eagle:footprint:6239920/1" value="5K" x="6.858" y="2.556" smashed="yes" rot="R90">
+<attribute name="MPN" value="0805W8F4871T5E" x="6.858" y="2.556" size="1.778" layer="27" rot="R90" display="off"/>
 <attribute name="NAME" x="5.572" y="1.524" size="0.8128" layer="25" rot="R180"/>
 <attribute name="VALUE" x="9.144" y="1.794" size="1.27" layer="27" rot="R90"/>

Commit message: fixed part number
Parts:
- U1: value AP211K-3.3 -> AP2112K-3.3
Changed lines of the file:
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@@
 <drawing>
 <settings>
-<setting alwaysvectorfont="yes"/>
+<setting alwaysvectorfont="no"/>
 <setting keepoldvectorfont="yes"/>
 <setting verticaltext="up"/>
@@
 </autorouter>
 <elements>
-<element name="U1" library="microbuilder" package="SOT23-5" value="AP211K-3.3" x="5.588" y="19.047" smashed="yes" rot="R90">
+<element name="U1" library="microbuilder" package="SOT23-5" value="AP2112K-3.3" x="5.588" y="19.047" smashed="yes" rot="R90">
 <attribute name="MPN" value="AP2112K-3.3" x="5.588" y="19.047" size="1.778" layer="27" rot="R90" display="off"/>
 <attribute name="NAME" x="5.21" y="16.764" size="0.8128" layer="25" rot="R180"/>

Commit message: renamed yellow led to white
Parts:
- CHG: value YELLOW -> WHITE
Changed lines of the file:
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@@
 <?xml version="1.0" encoding="utf-8"?>
 <!DOCTYPE eagle SYSTEM "eagle.dtd">
-<eagle version="9.6.2">
+<eagle version="9.5.0">
 <drawing>
 <settings>
@@
 </layers>
 <board>
-<fusionsync huburn="a.cGVyc29uYWw6dWUyODFhMTI5" projecturn="a.cGVyc29uYWw6dWUyODFhMTI5IzIwMTkwOTE3MjE1ODk1MzI2" f3durn="urn:adsk.wipprod:dm.lineage:P5lhZWs8S_KHtQ88bDf2NQ" pcbguid="cd0c53a3-0c54-43de-9435-58563155f29e" lastpulledtime="" lastsyncedchangeguid="89411407-e078-885e-39c3-f9a9a76d8070" latestrevisionid="" lastsyncedrevisionid="" lastboardhashguid="036b4d5f-3d3b-f5ef-ad34-bd3b1ec33525" lastpushedtime="2020-08-29T06:20:16Z" linktopcb3d="false"/>
+<fusionsync huburn="a.cGVyc29uYWw6dWUyODFhMTI5" projecturn="a.cGVyc29uYWw6dWUyODFhMTI5IzIwMTkwOTE3MjE1ODk1MzI2" f3durn="urn:adsk.wipprod:dm.lineage:P5lhZWs8S_KHtQ88bDf2NQ" pcbguid="cd0c53a3-0c54-43de-9435-58563155f29e" lastpulledtime="" lastsyncedchangeguid="89411407-e078-885e-39c3-f9a9a76d8070"/>
 <plain>
 <rectangle x1="44.831" y1="46.953" x2="45.339" y2="47.207" layer="42" rot="R90"/>
@@
 <attribute name="VALUE" x="21.336" y="18.615" size="0.4064" layer="27" ratio="10" rot="R90"/>
 </element>
-<element name="CHG" library="microbuilder" package="CHIPLED_0805_NOOUTLINE" value="YELLOW" x="19.304" y="2.54" smashed="yes" rot="MR0">
+<element name="CHG" library="microbuilder" package="CHIPLED_0805_NOOUTLINE" value="WHITE" x="19.304" y="2.54" smashed="yes" rot="MR0">
 <attribute name="MPN" value="NCD0805W2" x="19.304" y="2.54" size="1.778" layer="28" rot="MR0" display="off"/>
 <attribute name="NAME" x="20.193" y="4.572" size="0.8128" layer="26" ratio="18" rot="MR0"/>
