File: cad/pcb/oled.sch (EAGLE design)
At the start: 20 parts, among them U1 UG-2828GDEDF11, U2 FAN5331SX

Commit message: Revert "Revert OLED board to use 3.3V for input to the 13V FAN5331 boost"
This reverts commit 2f54354309870ccb091a2a633caf6ab9d6db30ca.
Connections:
- net +3V3: no longer C6.P$1, L1.1, U2.SHDN, U2.VIN
- net VIN: now also C6.P$1, L1.1, U2.SHDN, U2.VIN
Changed lines of the file:
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@@
 <attribute name="THRU-HOLE" value="1"/>
 </part>
-<part name="+3V1" library="supply1" library_urn="urn:adsk.eagle:library:371" deviceset="+3V3" device=""/>
+<part name="SUPPLY1" library="SparkFun-PowerSymbols" library_urn="urn:adsk.eagle:library:530" deviceset="VIN" device=""/>
 </parts>
 <sheets>
@@
 <attribute name="BOTTOM" x="215.9" y="93.98" size="1.778" layer="96" display="off"/>
 </instance>
-<instance part="+3V1" gate="G$1" x="193.04" y="180.34" smashed="yes">
-<attribute name="VALUE" x="191.516" y="181.356" size="1.27" layer="96"/>
+<instance part="SUPPLY1" gate="G$1" x="193.04" y="177.8" smashed="yes">
+<attribute name="VALUE" x="193.04" y="180.594" size="1.778" layer="96" align="bottom-center"/>
 </instance>
 </instances>
@@
 <pinref part="U1" gate="G$1" pin="VCI"/>
 </segment>
+</net>
+<net name="D1/GPIO5" class="0">
+<segment>
+<pinref part="JP1" gate="G$1" pin="3"/>
+<wire x1="213.36" y1="96.52" x2="203.2" y2="96.52" width="0.1524" layer="91"/>
+<label x="203.2" y="96.52" size="1.778" layer="95" rot="R180"/>
+</segment>
+</net>
+<net name="D2/GPIO4" class="0">
+<segment>
+<pinref part="JP1" gate="G$1" pin="4"/>
+<wire x1="213.36" y1="93.98" x2="203.2" y2="93.98" width="0.1524" layer="91"/>
+<label x="203.2" y="93.98" size="1.778" layer="95" rot="R180"/>
+</segment>
+</net>
+<net name="D3/GPIO0" class="0">
+<segment>
+<pinref part="JP1" gate="G$1" pin="5"/>
+<wire x1="213.36" y1="91.44" x2="203.2" y2="91.44" width="0.1524" layer="91"/>
+<label x="203.2" y="91.44" size="1.778" layer="95" rot="R180"/>
+</segment>
+</net>
+<net name="D4/GPIO2" class="0">
+<segment>
+<pinref part="JP1" gate="G$1" pin="6"/>
+<wire x1="213.36" y1="88.9" x2="203.2" y2="88.9" width="0.1524" layer="91"/>
+<label x="203.2" y="88.9" size="1.778" layer="95" rot="R180"/>
+</segment>
+<segment>
+<wire x1="129.54" y1="124.46" x2="111.76" y2="124.46" width="0.1524" layer="91"/>
+<label x="111.76" y="124.46" size="1.778" layer="95"/>
+<pinref part="U1" gate="G$1" pin="D/C#"/>
+</segment>
+</net>
+<net name="D8/GPIO15" class="0">
+<segment>
+<pinref part="JP2" gate="G$1" pin="2"/>
+<wire x1="228.6" y1="86.36" x2="238.76" y2="86.36" width="0.1524" layer="91"/>
+<label x="238.76" y="86.36" size="1.778" layer="95"/>
+</segment>
+<segment>
+<wire x1="129.54" y1="121.92" x2="111.76" y2="121.92" width="0.1524" layer="91"/>
+<label x="111.76" y="121.92" size="1.778" layer="95"/>
+<pinref part="U1" gate="G$1" pin="RES#"/>
+</segment>
+</net>
+<net name="D5/GPIO14/SCK" class="0">
+<segment>
+<pinref part="JP2" gate="G$1" pin="5"/>
+<wire x1="228.6" y1="93.98" x2="238.76" y2="93.98" width="0.1524" layer="91"/>
+<label x="238.76" y="93.98" size="1.778" layer="95"/>
+</segment>
+<segment>
+<wire x1="129.54" y1="139.7" x2="111.76" y2="139.7" width="0.1524" layer="91"/>
+<label x="111.76" y="139.7" size="1.778" layer="95"/>
+<pinref part="U1" gate="G$1" pin="D0/SCK"/>
+</segment>
+</net>
+<net name="D0/GPIO16" class="0">
+<segment>
+<pinref part="JP2" gate="G$1" pin="6"/>
+<wire x1="228.6" y1="96.52" x2="238.76" y2="96.52" width="0.1524" layer="91"/>
+<label x="238.76" y="96.52" size="1.778" layer="95"/>
+</segment>
+<segment>
+<wire x1="129.54" y1="127" x2="111.76" y2="127" width="0.1524" layer="91"/>
+<label x="111.76" y="127" size="1.778" layer="95"/>
+<pinref part="U1" gate="G$1" pin="CS#"/>
+</segment>
+</net>
+<net name="A0" class="0">
+<segment>
+<pinref part="JP2" gate="G$1" pin="7"/>
+<wire x1="228.6" y1="99.06" x2="238.76" y2="99.06" width="0.1524" layer="91"/>
+<label x="238.76" y="99.06" size="1.778" layer="95"/>
+</segment>
+</net>
+<net name="D7/GPIO13/MOSI" class="0">
+<segment>
+<pinref part="JP2" gate="G$1" pin="3"/>
+<wire x1="228.6" y1="88.9" x2="238.76" y2="88.9" width="0.1524" layer="91"/>
+<label x="238.76" y="88.9" size="1.778" layer="95"/>
+</segment>
+<segment>
+<wire x1="129.54" y1="142.24" x2="111.76" y2="142.24" width="0.1524" layer="91"/>
+<label x="111.76" y="142.24" size="1.778" layer="95"/>
+<pinref part="U1" gate="G$1" pin="D1/SDIN"/>
+</segment>
+</net>
+<net name="VIN" class="1">
 <segment>
 <wire x1="193.04" y1="167.64" x2="193.04" y2="160.02" width="0.1524" layer="91"/>
@@
 <pinref part="U2" gate="G$1" pin="SHDN"/>
 <pinref part="L1" gate="G$1" pin="1"/>
-<pinref part="+3V1" gate="G$1" pin="+3V3"/>
-</segment>
-</net>
-<net name="D1/GPIO5" class="0">
-<segment>
-<pinref part="JP1" gate="G$1" pin="3"/>
-<wire x1="213.36" y1="96.52" x2="203.2" y2="96.52" width="0.1524" layer="91"/>
-<label x="203.2" y="96.52" size="1.778" layer="95" rot="R180"/>
-</segment>
-</net>
-<net name="D2/GPIO4" class="0">
-<segment>
-<pinref part="JP1" gate="G$1" pin="4"/>
-<wire x1="213.36" y1="93.98" x2="203.2" y2="93.98" width="0.1524" layer="91"/>
-<label x="203.2" y="93.98" size="1.778" layer="95" rot="R180"/>
-</segment>
-</net>
-<net name="D3/GPIO0" class="0">
-<segment>
-<pinref part="JP1" gate="G$1" pin="5"/>
-<wire x1="213.36" y1="91.44" x2="203.2" y2="91.44" width="0.1524" layer="91"/>
-<label x="203.2" y="91.44" size="1.778" layer="95" rot="R180"/>
-</segment>
-</net>
-<net name="D4/GPIO2" class="0">
-<segment>
-<pinref part="JP1" gate="G$1" pin="6"/>
-<wire x1="213.36" y1="88.9" x2="203.2" y2="88.9" width="0.1524" layer="91"/>
-<label x="203.2" y="88.9" size="1.778" layer="95" rot="R180"/>
-</segment>
-<segment>
-<wire x1="129.54" y1="124.46" x2="111.76" y2="124.46" width="0.1524" layer="91"/>
-<label x="111.76" y="124.46" size="1.778" layer="95"/>
-<pinref part="U1" gate="G$1" pin="D/C#"/>
-</segment>
-</net>
-<net name="D8/GPIO15" class="0">
-<segment>
-<pinref part="JP2" gate="G$1" pin="2"/>
-<wire x1="228.6" y1="86.36" x2="238.76" y2="86.36" width="0.1524" layer="91"/>
-<label x="238.76" y="86.36" size="1.778" layer="95"/>
-</segment>
-<segment>
-<wire x1="129.54" y1="121.92" x2="111.76" y2="121.92" width="0.1524" layer="91"/>
-<label x="111.76" y="121.92" size="1.778" layer="95"/>
-<pinref part="U1" gate="G$1" pin="RES#"/>
-</segment>
-</net>
-<net name="D5/GPIO14/SCK" class="0">
-<segment>
-<pinref part="JP2" gate="G$1" pin="5"/>
-<wire x1="228.6" y1="93.98" x2="238.76" y2="93.98" width="0.1524" layer="91"/>
-<label x="238.76" y="93.98" size="1.778" layer="95"/>
-</segment>
-<segment>
-<wire x1="129.54" y1="139.7" x2="111.76" y2="139.7" width="0.1524" layer="91"/>
-<label x="111.76" y="139.7" size="1.778" layer="95"/>
-<pinref part="U1" gate="G$1" pin="D0/SCK"/>
-</segment>
-</net>
-<net name="D0/GPIO16" class="0">
-<segment>
-<pinref part="JP2" gate="G$1" pin="6"/>
-<wire x1="228.6" y1="96.52" x2="238.76" y2="96.52" width="0.1524" layer="91"/>
-<label x="238.76" y="96.52" size="1.778" layer="95"/>
-</segment>
-<segment>
-<wire x1="129.54" y1="127" x2="111.76" y2="127" width="0.1524" layer="91"/>
-<label x="111.76" y="127" size="1.778" layer="95"/>
-<pinref part="U1" gate="G$1" pin="CS#"/>
-</segment>
-</net>
-<net name="A0" class="0">
-<segment>
-<pinref part="JP2" gate="G$1" pin="7"/>
-<wire x1="228.6" y1="99.06" x2="238.76" y2="99.06" width="0.1524" layer="91"/>
-<label x="238.76" y="99.06" size="1.778" layer="95"/>
-</segment>
-</net>
-<net name="D7/GPIO13/MOSI" class="0">
-<segment>
-<pinref part="JP2" gate="G$1" pin="3"/>
-<wire x1="228.6" y1="88.9" x2="238.76" y2="88.9" width="0.1524" layer="91"/>
-<label x="238.76" y="88.9" size="1.778" layer="95"/>
-</segment>
-<segment>
-<wire x1="129.54" y1="142.24" x2="111.76" y2="142.24" width="0.1524" layer="91"/>
-<label x="111.76" y="142.24" size="1.778" layer="95"/>
-<pinref part="U1" gate="G$1" pin="D1/SDIN"/>
-</segment>
-</net>
-<net name="VIN" class="1">
+<pinref part="SUPPLY1" gate="G$1" pin="VIN"/>
+</segment>
 <segment>
 <pinref part="JP1" gate="G$1" pin="8"/>

Commit message: replace C2,C3,C4,C6 on oled board with CL21A106KOQNNNE (10uF,16V)
Parts:
- C2, C3, C4, C6: MPN LMK212BJ106KG-T -> CL21A106KOQNNNE
Changed lines of the file:
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@@
 <?xml version="1.0" encoding="utf-8"?>
 <!DOCTYPE eagle SYSTEM "eagle.dtd">
-<eagle version="9.5.0">
+<eagle version="9.6.2">
 <drawing>
 <settings>
@@
 </part>
 <part name="C2" library="microbuilder" deviceset="CAP_CERAMIC" device="0805" override_package3d_urn="urn:adsk.eagle:package:21520266/2" override_package_urn="urn:adsk.eagle:footprint:21520267/1" value="10uF/16V">
-<attribute name="MPN" value="LMK212BJ106KG-T"/>
+<attribute name="MPN" value="CL21A106KOQNNNE"/>
 </part>
 <part name="C5" library="microbuilder" deviceset="CAP_CERAMIC" device="0805" override_package3d_urn="urn:adsk.eagle:package:21520244/3" override_package_urn="urn:adsk.eagle:footprint:21520245/1" value="1.0uF">
@@
 </part>
 <part name="C3" library="microbuilder" deviceset="CAP_CERAMIC" device="0805" override_package3d_urn="urn:adsk.eagle:package:21519624/2" override_package_urn="urn:adsk.eagle:footprint:21519625/1" value="10uF">
-<attribute name="MPN" value="LMK212BJ106KG-T"/>
+<attribute name="MPN" value="CL21A106KOQNNNE"/>
 </part>
 <part name="GND1" library="supply1" library_urn="urn:adsk.eagle:library:371" deviceset="GND" device=""/>
@@
 </part>
 <part name="C6" library="microbuilder" deviceset="CAP_CERAMIC" device="0805" override_package3d_urn="urn:adsk.eagle:package:21520293/2" override_package_urn="urn:adsk.eagle:footprint:21520294/1" value="10uF">
-<attribute name="MPN" value="LMK212BJ106KG-T"/>
+<attribute name="MPN" value="CL21A106KOQNNNE"/>
 </part>
 <part name="L1" library="microbuilder" deviceset="INDUCTOR" device="" value="10uH">
@@
 </part>
 <part name="C4" library="microbuilder" deviceset="CAP_CERAMIC" device="0805" override_package3d_urn="urn:adsk.eagle:package:21520257/2" override_package_urn="urn:adsk.eagle:footprint:21520262/1" value="10uF/16V">
-<attribute name="MPN" value="LMK212BJ106KG-T"/>
+<attribute name="MPN" value="CL21A106KOQNNNE"/>
 </part>
 <part name="D1" library="microbuilder" deviceset="DIODE" device="SOD-323" value="1N4148">
